File: fonte 12v/fonte 12v.kicad_sch (KiCad schematic)
At the start: 4 parts

Commit message: modificação esquematico
Parts:
- added D1: ABS2, Diode_SMD:Diode_Bridge_Diotec_ABS, symbol Diode_Bridge:ABS2
- FL1: value Choke_Schaffner_RN102-0.3-02-12M -> ~
Connections:
- net AC: now also FL1.1
- net at CX1.2, F1.2, R25.2: now also FL1.3; no longer FL1.2
Other:
- moved on the sheet: FL1
Changed lines of the file:
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@@
 	(paper "A4")
+	(junction
+		(at 29.21 63.5)
+		(diameter 0)
+		(color 0 0 0 0)
+	)
 	(junction
 		(at 29.21 50.8)
@@
 	)
 	(junction
-		(at 33.02 63.5)
+		(at 44.45 63.5)
 		(diameter 0)
 		(color 0 0 0 0)
@@
 	(wire
 		(pts
+			(xy 44.45 73.66) (xy 44.45 63.5)
+		)
+		(stroke
+			(width 0)
+			(type default)
+		)
+	)
+	(wire
+		(pts
 			(xy 29.21 41.91) (xy 29.21 50.8)
 		)
@@
 	(wire
 		(pts
+			(xy 39.37 73.66) (xy 44.45 73.66)
+		)
+		(stroke
+			(width 0)
+			(type default)
+		)
+	)
+	(wire
+		(pts
 			(xy 44.45 50.8) (xy 40.64 50.8)
 		)
@@
 	(wire
 		(pts
+			(xy 29.21 73.66) (xy 34.29 73.66)
+		)
+		(stroke
+			(width 0)
+			(type default)
+		)
+	)
+	(wire
+		(pts
 			(xy 44.45 63.5) (xy 44.45 50.8)
 		)
@@
 	(wire
 		(pts
-			(xy 34.29 73.66) (xy 34.29 63.5)
+			(xy 29.21 73.66) (xy 29.21 63.5)
 		)
 		(stroke
@@
 		(pts
 			(xy 29.21 25.4) (xy 29.21 34.29)
-		)
-		(stroke
-			(width 0)
-			(type default)
-		)
-	)
-	(wire
-		(pts
-			(xy 33.02 63.5) (xy 34.29 63.5)
 		)
 		(stroke
@@
 	(symbol
 		(lib_id "Filter:Choke_Schaffner_RN102-0.3-02-12M")
-		(at 36.83 78.74 90)
+		(at 36.83 78.74 270)
 		(unit 1)
 		(exclude_from_sim no)
@@
 		(fields_autoplaced yes)
 		(property "Reference" "FL1"
-			(at 40.64 77.8509 90)
-			(effects
-				(font
-					(size 1.27 1.27)
-				)
-				(justify right)
-			)
-		)
-		(property "Value" "Choke_Schaffner_RN102-0.3-02-12M"
-			(at 40.64 80.3909 90)
-			(effects
-				(font
-					(size 1.27 1.27)
-				)
-				(justify right)
+			(at 40.64 77.7239 90)
+			(effects
+				(font
+					(size 1.27 1.27)
+				)
+				(justify left)
+			)
+		)
+		(property "Value" "~"
+			(at 40.64 79.629 90)
+			(effects
+				(font
+					(size 1.27 1.27)
+				)
+				(justify left)
 			)
 		)
@@
 					(unit 1)
 				)
+			)
+		)
+	)
+	(symbol
+		(lib_id "Diode_Bridge:ABS2")
+		(at 39.37 99.06 0)
+		(unit 1)
+		(exclude_from_sim no)
+		(in_bom yes)
+		(on_board yes)
+		(dnp no)
+		(fields_autoplaced yes)
+		(property "Reference" "D1"
+			(at 48.26 92.6398 0)
+			(effects
+				(font
+					(size 1.27 1.27)
+				)
+			)
+		)
+		(property "Value" "ABS2"
+			(at 48.26 95.1798 0)
+			(effects
+				(font
+					(size 1.27 1.27)
+				)
+			)
+		)
+		(property "Footprint" "Diode_SMD:Diode_Bridge_Diotec_ABS"
+			(at 43.18 95.885 0)
+			(effects
+				(font
+					(size 1.27 1.27)
+				)
+				(justify left)
+				(hide yes)
+			)
+		)
+		(property "Datasheet" "https://diotec.com/tl_files/diotec/files/pdf/datasheets/abs2.pdf"
+			(at 39.37 99.06 0)
+			(effects
+				(font
+					(size 1.27 1.27)
+				)
+				(hide yes)
+			)
+		)
+		(property "Description" "Miniature Glass Passivated Single-Phase Surface Mount Bridge Rectifiers, 140V Vrms, 0.8A If, ABS SMD package"
+			(at 39.37 99.06 0)
+			(effects
+				(font
+					(size 1.27 1.27)
+				)
+				(hide yes)
+			)
+		)
+		(pin "3"
+		)
+		(pin "2"
+		)
+		(pin "1"
+		)
+		(pin "4"
+		)
+		(instances
+			(project ""
+				(path "/350fa56d-c7dc-4741-86f8-d85412a3873b"
+					(reference "D1")
+					(unit 1)
+				)

Commit message: atualizacao esquematico
Parts:
- removed D1: ABS2, Diode_SMD:Diode_Bridge_Diotec_ABS, symbol Diode_Bridge:ABS2
- added C1, C2: C, symbol Device:C
- added C3: C_Polarized, symbol Device:C_Polarized
- added D1: RB151, Diode_THT:Diode_Bridge_Round_D9.0mm, symbol Diode_Bridge:RB151
- added D2: D, symbol Device:D
- added JP1: Jumper_2_Bridged, symbol Jumper:Jumper_2_Bridged
- added Q1: BC107, Package_TO_SOT_THT:TO-18-3, symbol Transistor_BJT:BC107
- added R1, R2, R3: R, symbol Device:R
Connections:
- net Earth: now also C1.2, C2.2
- net at FL1.2: now also C2.1, D1.4
- net at FL1.4: now also C1.1, D1.2
- new net: C3.1, D1.1 (+)
- new net: C3.2, D1.3 (-), JP1.1 (A), R1.1, R2.1
- new net: D2.2 (A), R1.2, R3.1

Commit message: atualizado esquematico
Parts:
- C1: renamed from C3; value C_Polarized -> 100 μF
- C12: renamed from C1; value C -> 3.56 nF
- C13: renamed from C2; value C -> 3.57 nF
- D1: value RB151 -> ~
- R13: renamed from R3; value R -> 33 Ω
- R14: renamed from R1; value R -> 20k Ω
Other:
- moved on the sheet: D2
Changed lines of the file:
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@@
 	(wire
 		(pts
-			(xy 96.52 113.03) (xy 104.14 113.03)
+			(xy 96.52 113.03) (xy 106.68 113.03)
 		)
 		(stroke
@@
 		(fields_autoplaced yes)
 		(property "Reference" "D1"
-			(at 48.26 114.2298 90)
-			(effects
-				(font
-					(size 1.27 1.27)
-				)
-			)
-		)
-		(property "Value" "RB151"
-			(at 48.26 116.7698 90)
+			(at 45.72 114.2298 90)
+			(effects
+				(font
+					(size 1.27 1.27)
+				)
+			)
+		)
+		(property "Value" "~"
+			(at 45.72 116.7698 90)
 			(effects
 				(font
@@
 	(symbol
 		(lib_id "Device:D")
-		(at 104.14 116.84 90)
+		(at 106.68 116.84 90)
 		(unit 1)
 		(exclude_from_sim no)
@@
 		(fields_autoplaced yes)
 		(property "Reference" "D2"
-			(at 106.68 115.5699 90)
+			(at 109.22 115.5699 90)
 			(effects
 				(font
@@
 		)
 		(property "Value" "D"
-			(at 106.68 118.1099 90)
+			(at 109.22 118.1099 90)
 			(effects
 				(font
@@
 		)
 		(property "Footprint" ""
-			(at 104.14 116.84 0)
-			(effects
-				(font
-					(size 1.27 1.27)
-				)
-				(hide yes)
-			)
-		)
-		(property "Datasheet" "~"
-			(at 104.14 116.84 0)
+			(at 106.68 116.84 0)
+			(effects
+				(font
+					(size 1.27 1.27)
+				)
+				(hide yes)
+			)
+		)
+		(property "Datasheet" "~"
+			(at 106.68 116.84 0)
 			(effects
 				(font
@@
 		)
 		(property "Description" "Diode"
-			(at 104.14 116.84 0)
+			(at 106.68 116.84 0)
 			(effects
 				(font
@@
 		)
 		(property "Sim.Device" "D"
-			(at 104.14 116.84 0)
+			(at 106.68 116.84 0)
 			(effects
 				(font
@@
 		)
 		(property "Sim.Pins" "1=K 2=A"
-			(at 104.14 116.84 0)
+			(at 106.68 116.84 0)
 			(effects
 				(font
@@
 		(dnp no)
 		(fields_autoplaced yes)
-		(property "Reference" "C3"
+		(property "Reference" "C1"
 			(at 66.04 120.2689 0)
 			(effects
@@
 			)
 		)
-		(property "Value" "C_Polarized"
+		(property "Value" "100 μF"
 			(at 66.04 122.8089 0)
 			(effects
@@
 			(project ""
 				(path "/350fa56d-c7dc-4741-86f8-d85412a3873b"
-					(reference "C3")
+					(reference "C1")
 					(unit 1)
 				)
@@
 		(dnp no)
 		(fields_autoplaced yes)
-		(property "Reference" "R1"
+		(property "Reference" "R14"
 			(at 86.36 106.68 90)
 			(effects
@@
 			)
 		)
-		(property "Value" "R"
+		(property "Value" "20k Ω"
 			(at 86.36 109.22 90)
 			(effects
@@
 			(project ""
 				(path "/350fa56d-c7dc-4741-86f8-d85412a3873b"
-					(reference "R1")
+					(reference "R14")
 					(unit 1)
 				)
@@
 		(dnp no)
 		(fields_autoplaced yes)
-		(property "Reference" "C1"
+		(property "Reference" "C12"
 			(at 38.1 92.7099 0)
 			(effects
@@
 			)
 		)
-		(property "Value" "C"
+		(property "Value" "3.56 nF"
 			(at 38.1 95.2499 0)
 			(effects
@@
 			(project ""
 				(path "/350fa56d-c7dc-4741-86f8-d85412a3873b"
-					(reference "C1")
+					(reference "C12")
 					(unit 1)
 				)
@@
 		(dnp no)
 		(fields_autoplaced yes)
-		(property "Reference" "R3"
+		(property "Reference" "R13"
 			(at 99.06 115.5699 0)
 			(effects
@@
 			)
 		)
-		(property "Value" "R"
+		(property "Value" "33 Ω"
 			(at 99.06 118.1099 0)
 			(effects
@@
 			(project "fonte 12v"
 				(path "/350fa56d-c7dc-4741-86f8-d85412a3873b"
-					(reference "R3")
+					(reference "R13")
 					(unit 1)
 				)
@@
 		(dnp no)
 		(fields_autoplaced yes)
-		(property "Reference" "C2"
+		(property "Reference" "C13"
 			(at 46.99 92.7099 0)
 			(effects
@@
 			)
 		)
-		(property "Value" "C"
+		(property "Value" "3.57 nF"
 			(at 46.99 95.2499 0)
 			(effects
@@
 			(project ""
 				(path "/350fa56d-c7dc-4741-86f8-d85412a3873b"
-					(reference "C2")
-					(unit 1)
-				)
+					(reference "C13")
+					(unit 1)
+				)
